Commit message: rviz and motor control

File: warehousebot_description/urdf/warehousebot.urdf (robot description, URDF)
Before this commit: robot warehousebot, 3 links, 2 joints
Links:
- link base_link: geometry visual mesh filename=package://warehousebot_description/meshes/body.dae scale=5 5 5
Joints:
- joint lidar_joint: origin xyz=0.0 0.0 0.42 rpy=0 0 0 -> xyz=0.0 0.0 0.55 rpy=0 0 0
- joint scissor_joint: origin xyz= 0.0 -0.5 0.7 rpy=0 0 0 -> xyz= 0.0 -0.65 0.9 rpy=0 0 0

Commit message: Working ST Motor Controller implementation

File: warehousebot_description/urdf/warehousebot.urdf (robot description, URDF)
Before this commit: robot warehousebot, 3 links, 2 joints
Links:
- link base_link: geometry visual mesh filename=package://warehousebot_description/meshes/body_1.dae scale=5 5 5

Commit message: teleop and base modify

File: warehousebot_description/urdf/warehousebot.urdf (robot description, URDF)
Before this commit: robot warehousebot, 3 links, 2 joints
Links:
- removed link scissor_link
- link base_link: geometry visual mesh filename=package://warehousebot_description/meshes/mob_base.dae scale=5 5 5
- link rplidar_link: geometry visual cylinder length=0.08 radius=0.08
Joints:
- removed joint scissor_joint
- joint lidar_joint: origin xyz=0.0 0.0 0.55 rpy=0 0 0 -> xyz=0.0 0.25 0.3 rpy=0 0 0

Commit message: test control teb from laptop config

File: warehousebot_description/urdf/warehousebot.urdf (robot description, URDF)
Before this commit: robot warehousebot, 2 links, 1 joints
Links:
- removed link rplidar_link
- added link laser; visual cylinder length=0.08 radius=0.08
Joints:
- removed joint lidar_joint
- added joint laser_join: type fixed, parent base_link, child laser, origin xyz=0.0 0.25 0.3 rpy=0 0 0
